File: kicad/c34/c34.kicad_sch (KiCad schematic)
At the start: 14 parts, among them K1 SANYOU_SRD_Form_C, Q1 TRANS_NPN-MMBT2222AL, SW1 SW_Push, U1 MOUDLE-SEEEDUINO-XIAO-ESP32C3

Commit message: Update c34.kicad_sch
Parts:
- R2: value 10k -> 1k
Changed lines of the file:
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@@
 			)
 		)
-		(property "Value" "10k"
+		(property "Value" "1k"
 			(at 215.9 135.89 90)
 			(effects
